Commit message: Modified to work with KDL planner

File: stretch_description/urdf/stretch_main.xacro (robot description, xacro)
@@ -8,5 +8,5 @@
   <link
     name="base_link">
-    <inertial>
+    <!-- <inertial>
       <origin
         xyz="-0.109461304328163 -0.000741018909047708 0.0914915269429946"
@@ -21,5 +21,5 @@
         iyz="1.33487716258445E-05"
         izz="0.0037204727467362" />
-    </inertial>
+    </inertial> -->
     <visual>
       <origin
